File: kicad/kint.kicad_sch (KiCad schematic)
At the start: 25 parts, among them J1 THUMB_RIGHT_SPC_KB600, J2 LEFT_13_LT, J3 TOP_LEFT, J4 TOP_RIGHT, J5 THUMB_LEFT_BAK, J6 THUMB_RIGHT_SPC, J7 RIGHT_13_DOWN, J8 THUMB_LEFT_BAK_KB600, U1 TEENSY_3.5_3.6

Commit message: initial commit of kinesis2040
Parts:
- removed JP1, JP2, JP3: SolderJumper_2_Open, Jumper:SolderJumper-2_P1.3mm_Open_RoundedPad1.0x1.5mm, symbol Jumper:SolderJumper_2_Open
- removed JP4, JP5, JP6: SolderJumper_2_Bridged, Jumper:SolderJumper-2_P1.3mm_Bridged2Bar_RoundedPad1.0x1.5mm, symbol Jumper:SolderJumper_2_Bridged
- removed LED1, LED2, LED3, LED4: LEDSML1206, LED_SMD:LED_1206_3216Metric_Pad1.42x1.75mm_HandSolder, symbol Device:LED
- removed R1, R2, R3, R4: 10K, Resistor_SMD:R_1206_3216Metric_Pad1.42x1.75mm_HandSolder, symbol Device:R
- J1, J2, J3, J4, J5, J6, J7, J8: MPN 39-53-2135 -> (none); digikeypn WM14526-ND -> (none); mouserpn 538-39-53-2135 -> (none)
Connections:
- net 3V3: now also U1.3.3V; no longer U1.3V3_2
- net COL_0: now also U1.GPIO27/ADC1/I2C_SCL; no longer U1.18/A4/SDA
- net COL_1: now also U1.GPIO23; no longer U1.14/A0
- net COL_2: now also U1.GPIO12/SPI1_RX/I2C0_SDA/UART0_TX, U1.GPIO20/I2C0_SDA
- net COL_3: now also U1.GPIO29/ADC3; no longer U1.20/A6
- net COL_4: now also U1.GPIO18; no longer U1.22/A8
- net COL_5: now also U1.GPIO28/ADC2; no longer U1.19/A5/SCL
- net COL_6: now also U1.GPIO03/SPI0_TX/I2C_SCL; no longer U1.6
- net GND: no longer U1.GND, U1.GND3
- net ROW_0: now also U1.GPIO18/SPI0_SCK/I2C0_SDA; no longer U1.0/RX
- net ROW_1: now also U1.GPIO06/SPI0_SCK/I2C1_SDA; no longer U1.9/CS
- net ROW_2: now also U1.GPIO07/SPI0_TX/I2C1_SCL; no longer U1.10/CS
- net ROW_3: now also U1.GPIO08/SPI1_RX/I2C0_SDA/UART1_TX; no longer U1.11/MOSI
- net ROW_4: now also U1.GPIO04/SPI0_RX/I2C0_SDA/UART1_TX, U1.GPIO09/SPI1_CSn/I2C0_SCL/UART1_RX
- net ROW_5: now also U1.GPIO21/I2C0_SCL, U1.GPIO22
- net ROW_6: now also U1.GPIO02/SPI0_SCK/I2C1_SDA; no longer U1.5
- net ROW_7: now also U1.GPIO00/SPI0_RX/I2C0_SDA/UART0_TX; no longer U1.3/CANTX
- net ROW_8: now also U1.GPIO01/SPI0_CSn/I2C0_SCL/UART0_RX; no longer U1.4/CANRX
- net ROW_9: now also U1.GPIO25/SPI0_CSn/I2C0_SCL/UART0_RX; no longer U1.1/TX
- net ROW_EQL: now also U1.GPIO05/SPI0_CSn/I2C0_SCL/UART1_RX; no longer U1.8
- net ROW_ESC: now also U1.GPIO26/ADC0/I2C1_SDA; no longer U1.17/A3
- net ROW_F1: now also U1.GPIO24; no longer U1.23/A9
- net ROW_F2: now also U1.GPIO11; no longer U1.21/A7
- net ROW_MIN: now also U1.GPIO10/SPI1_SCK/I2C1_SDA; no longer U1.2
- removed net LED_CAPS_LOCK: U1.12/MISO
- removed net LED_KEYPAD: U1.24
- removed net LED_NUM_LOCK: U1.26
- removed net LED_SCROLL_LOCK: U1.25
- no-connect marks 52 -> 31
Other:
- note removed: "TEENSY_POWER_LED"
- note removed: "Teensy++"
- note removed: "only present on: Teensy 3.5 Teensy 3.6 Teensy 4.1"
- company: Michael Stapelberg -> Fritz
- title: kinT keyboard controller -> kinesis2040 keyboard controller
